File: PCB/aeris/aeris.kicad_sch (KiCad schematic)
At the start: 13 parts, among them J1 SHT45, J2 LPS22HB, J3 SCD40, J4 SGP41, U3 ESP32-H2-SUPERMINI

Commit message: Update PCB
Parts:
- added C3, C4, C5, C6, C7, C8, C9: 0.1µF, Capacitor_SMD:C_1206_3216Metric, symbol Device:C
- added J5: PMSA003A, symbol Connector_Generic:Conn_02x05_Odd_Even
- added R1, R2: 10K, symbol Device:R
- added U1: 74AHCT244, symbol 74xx:74AHCT244
Connections:
- net +3V3: now also R1.2, R2.2
- net +5V: now also D1.4 (VDD), D2.4 (VDD), D3.4 (VDD), D4.4 (VDD), D5.4 (VDD), D6.4 (VDD), C3.1, C4.1, C5.1, C6.1, C7.1, C8.1, C9.1, J5.1 (Pin_1), J5.2 (Pin_2), U1.20 (VCC)
- net GND: now also D1.2 (VSS), D2.2 (VSS), D3.2 (VSS), D4.2 (VSS), D5.2 (VSS), D6.2 (VSS), C3.2, C4.2, C5.2, C6.2, C7.2, C8.2, C9.2, J5.3 (Pin_3), J5.4 (Pin_4), U1.1 (1OE), U1.10 (GND), U1.19 (2OE)
- net GPIO2: now also J5.5 (Pin_5), R1.1
- net GPIO22: now also D1.3 (DIN), D2.3 (DIN), D3.3 (DIN), D4.3 (DIN), D5.3 (DIN), D6.3 (DIN), J5.9 (Pin_9), U1.12 (1Y3), U1.14 (1Y2), U1.15 (2A1), U1.16 (1Y1), U1.17 (2A0), U1.18 (1Y0), U1.2 (1A0), U1.3 (2Y0), U1.4 (1A1), U1.5 (2Y1), U1.6 (1A2), U1.8 (1A3)
- net GPIO23: now also J5.10 (Pin_10), R2.1
- net GPIO24: now also J5.6 (Pin_6)
- no-connect marks 2 -> 14
Other:
- note added: "PLANTOWER PMSA003-A"
- moved on the sheet: D1, D2, D3, D4, D5, D6

Commit message: Update PCB
Parts:
- added Q1: BSS138, Package_TO_SOT_SMD:SOT-23, symbol Transistor_FET:BSS138
- added R3, R4: 10K, symbol Device:R
- added R5: 75R, symbol Device:R
